File: Carrier-Board-Mirroredv2/Carrier-Board.kicad_pcb (KiCad board)
At the start: 4 copper layers, 92 x 96 mm, 115 parts, among them J1 CONN_3-6318491-6, J10 Conn_02x03_Odd_Even, J2 Conn_01x0, J4 SI-51009-F, J6 Conn_01x03_Male, J7 Conn_01x03_Male, J8 Conn_01x06_Male, J9 Conn_02x04_Odd_Even, SW1 SW_Push, SW2 SW_Push, SW3 SW_Push, U1 MPM3620, U2 MPM3620, m1 MountingHole_2.7mm_M2.5_Pad, m2 MountingHole_2.7mm_M2.5_Pad

Commit message: Revised Mirrored Board
Complete mirrored board with traces (Minus micro USB port)
Parts:
- removed the ? at (21.4, 224.7)
- removed the ? at (19.4, 115.9)
- removed the C1 at (229.4, 67.9)
- removed the C1 at (61.5, 100.6)
- removed the C2 at (233.4, 69.4)
- removed the C2 at (63.0, 104.6)
- removed the C27 at (211.8, 58.6)
- removed the C27 at (96.7, 75.2)
- removed the C28 at (205.1, 58.5)
- removed the C28 at (96.7, 68.4)
- removed the C29 at (192.8, 57.9)
- removed the C29 at (97.3, 56.2)
- removed the C3 at (223.6, 79.8)
- removed the C3 at (73.4, 94.8)
- removed the C4 at (227.4, 81.1)
- removed the C4 at (74.7, 98.5)
- removed the D5 at (235.1, 76.5)
- removed the D5 at (70.1, 106.3)
- removed the D6 at (237.7, 78.9)
- removed the D6 at (72.5, 108.9)
- removed the D7 at (237.8, 81.7)
- removed the D7 at (75.3, 108.9)
- removed the D8 at (237.8, 84.5)
- removed the D8 at (78.1, 108.9)
- removed the G1 at (236.8, 110.1)
- removed the G1 at (208.8, 42.6)
- removed the G1 at (61.1, 89.6)
- removed the G1 at (62.1, 66.1)
- removed the J1 at (173.0, 95.7)
- removed the J1 at (98.9, 44.4)
- removed the J10 at (224.4, 115.0)
- removed the J10 at (23.0, 81.2)
- removed the J2 at (233.9, 50.9)
- removed the J2 at (42.8, 104.2)
- removed the J3 at (208.5, 30.7)
- removed the J3 at (63.5, 26.3)
- removed the J4 at (155.4, 72.1)
- removed the J4 at (91.0, 121.1)
- removed the J5 at (208.5, 35.7)
- removed the J5 at (63.5, 31.4)
- removed the J6 at (199.7, 114.9)
- removed the J6 at (105.7, 45.1)
- removed the J7 at (190.5, 115.0)
- removed the J7 at (22.8, 69.7)
- removed the J8 at (215.9, 114.5)
- removed the J8 at (21.0, 61.5)
- removed the J9 at (181.3, 115.4)
- removed the J9 at (23.2, 92.6)
- removed the R1 at (237.2, 69.4)
- removed the R1 at (63.0, 108.3)
- removed the R10 at (183.2, 76.7)
- removed the R10 at (96.3, 93.0)
- removed the R11 at (248.6, 26.7)
- removed the R11 at (23.0, 22.5)
- removed the R12 at (246.7, 32.9)
- removed the R12 at (24.9, 28.7)
- removed the R13 at (246.7, 36.7)
- removed the R13 at (24.9, 32.4)
- removed the R2 at (238.2, 66.2)
- removed the R2 at (59.8, 109.3)
- removed the R23 at (238.5, 81.6)
- removed the R23 at (75.2, 109.6)
- removed the R24 at (238.4, 79.2)
- removed the R24 at (72.8, 109.5)
- removed the R25 at (238.5, 84.6)
- removed the R25 at (78.2, 109.6)
- removed the R3 at (228.7, 63.9)
- removed the R3 at (57.5, 99.8)
- removed the R32 at (213.3, 51.0)
- removed the R32 at (104.2, 76.6)
- removed the R4 at (232.4, 60.9)
- removed the R4 at (54.5, 103.6)
- removed the R5 at (231.6, 80.8)
- removed the R5 at (74.4, 102.8)
- removed the R6 at (231.6, 77.3)
- removed the R6 at (70.9, 102.8)
- removed the R7 at (223.3, 75.8)
- removed the R7 at (69.4, 94.5)
- removed the R8 at (226.6, 73.1)
- removed the R8 at (66.7, 97.8)
- removed the R9 at (183.7, 67.3)
- removed the R9 at (86.8, 92.6)
- removed the REF** at (171.6, 29.4)
- removed the REF** at (26.6, 25.0)
- removed the REF** at (22.8, 110.7)
- removed the REF** at (102.8, 110.7)
- removed the REF** at (100.3, 25.0)
- removed the REF** at (52.8, 79.9)
- removed the REF** at (212.3, 83.9)
- removed the REF** at (194.5, 83.9)
- removed the REF** at (245.3, 29.3)
- removed the REF** at (203.4, 83.9)
- removed the REF** at (104.8, 219.5)
- removed the REF** at (24.8, 219.5)
- removed the REF** at (70.6, 79.9)
- removed the REF** at (61.7, 79.9)
- removed the SW1 at (249.3, 27.0)
- removed the SW1 at (22.3, 22.8)
- removed the SW2 at (249.2, 31.7)
- removed the SW2 at (22.4, 27.5)
- removed the SW3 at (249.2, 36.5)
- removed the SW3 at (22.4, 32.3)
- removed the U1 at (233.9, 64.9)
- removed the U1 at (58.5, 105.1)
- removed the U2 at (227.9, 76.8)
- removed the U2 at (70.4, 99.1)
- removed the U9 at (190.5, 58.3)
- removed the U9 at (96.8, 53.7)
- removed the m1 at (249.1, 53.4)
- removed the m1 at (249.1, 100.4)
- added ?: pc104, Carrier-Board:pc104, F.Cu at (25.4, 121.3)
- added C1: 10uF, Capacitors_SMD:C_0805, F.Cu at (67.6, 106.0)
- added C1: 10uF, Capacitors_SMD:C_0805, B.Cu at (210.6, 80.2)
- added C2: 22uF, Capacitors_SMD:C_0805, F.Cu at (69.1, 110.0)
- added C2: 22uF, Capacitors_SMD:C_0805, B.Cu at (209.1, 84.2)
- added C27: .1uF, Capacitors_SMD:C_0603, F.Cu at (102.7, 80.5)
- added C27: .1uF, Capacitors_SMD:C_0603, F.Cu at (226.2, 77.5)
- added C28: .1uF, Capacitors_SMD:C_0603, F.Cu at (102.7, 73.8)
- added C28: .1uF, Capacitors_SMD:C_0603, F.Cu at (226.3, 70.8)
- added C29: .1uF, Capacitors_SMD:C_0603, F.Cu at (103.3, 61.5)
- added C29: .1uF, Capacitors_SMD:C_0603, F.Cu at (226.9, 58.5)
- added C3: 10uF, Capacitors_SMD:C_0805, F.Cu at (79.5, 100.2)
- added C3: 10uF, Capacitors_SMD:C_0805, B.Cu at (198.7, 74.4)
- added C4: 22uF, Capacitors_SMD:C_0805, F.Cu at (80.7, 103.9)
- added C4: 22uF, Capacitors_SMD:C_0805, B.Cu at (197.4, 78.1)
- added D5: D_Zener 9V, Diodes_SMD:D_SOD-323, B.Cu at (76.1, 111.7)
- added D5: D_Zener 9V, Diodes_SMD:D_SOD-323, F.Cu at (202.0, 85.9)
- added D6: LED, Diodes_SMD:D_1206, F.Cu at (78.6, 114.2)
- added D6: LED, Diodes_SMD:D_1206, B.Cu at (199.6, 88.5)
- added D7: LED, Diodes_SMD:D_1206, F.Cu at (81.4, 114.3)
- added D7: LED, Diodes_SMD:D_1206, B.Cu at (196.8, 88.5)
- added D8: LED, Diodes_SMD:D_1206, F.Cu at (84.2, 114.3)
- added D8: LED, Diodes_SMD:D_1206, B.Cu at (194.0, 88.5)
- added G1: LOGO, BusSimulator:LetSatLogo440, F.Cu at (68.1, 71.5)
- added G1: LOGO, BusSimulator:LetSatLogo440, B.Cu at (67.1, 95.0)
- added G1: LOGO, BusSimulator:LetSatLogo440, F.Cu at (200.8, 67.2)
- added G1: LOGO, BusSimulator:LetSatLogo440, B.Cu at (174.8, 94.3)
- added J1: CONN_3-6318491-6, BusSimulator:ComExpressMini10, F.Cu at (105.0, 49.8)
- added J1: CONN_3-6318491-6, BusSimulator:ComExpressMini10, F.Cu at (228.5, 46.7)
- added J10: Conn_02x03_Odd_Even, Pin_Headers:Pin_Header_Angled_2x03_Pitch2.54mm, F.Cu at (29.1, 86.5)
- added J10: Conn_02x03_Odd_Even, Pin_Headers:Pin_Header_Angled_2x03_Pitch2.54mm, F.Cu at (152.5, 83.5)
- added J2: Conn_01x0, Connectors:Barrel_Jack_CUI_PJ-036AH-SMT, F.Cu at (48.9, 109.6)
- added J2: Conn_01x0, Connectors:Barrel_Jack_CUI_PJ-036AH-SMT, B.Cu at (179.2, 80.6)
- added J3: , Carrier-Board:ESQ-126-XX-X-D, F.Cu at (69.5, 31.7)
- added J3: , Carrier-Board:ESQ-126-XX-X-D, B.Cu at (194.4, 28.7)
- added J4: SI-51009-F, Carrier-Board:SI-51009-F, F.Cu at (97.0, 126.5)
- added J4: SI-51009-F, Carrier-Board:SI-51009-F, B.Cu at (224.2, 124.4)
- added J5: , Carrier-Board:ESQ-126-XX-X-D, F.Cu at (69.5, 36.8)
- added J5: , Carrier-Board:ESQ-126-XX-X-D, B.Cu at (194.4, 33.7)
- added J6: Conn_01x03_Male, Pin_Headers:Pin_Header_Angled_1x03_Pitch2.54mm, F.Cu at (111.7, 50.5)
- added J6: Conn_01x03_Male, Pin_Headers:Pin_Header_Angled_1x03_Pitch2.54mm, F.Cu at (235.2, 47.4)
- added J7: Conn_01x03_Male, Pin_Headers:Pin_Header_Angled_1x03_Pitch2.54mm, F.Cu at (28.8, 75.1)
- added J7: Conn_01x03_Male, Pin_Headers:Pin_Header_Angled_1x03_Pitch2.54mm, F.Cu at (152.3, 72.1)
- added J8: Conn_01x06_Male, Pin_Headers:Pin_Header_Angled_1x06_Pitch2.54mm, F.Cu at (27.0, 66.8)
- added J8: Conn_01x06_Male, Pin_Headers:Pin_Header_Angled_1x06_Pitch2.54mm, F.Cu at (150.5, 63.8)
- added J9: Conn_02x04_Odd_Even, Pin_Headers:Pin_Header_Angled_2x04_Pitch2.54mm, F.Cu at (29.3, 98.0)
- added J9: Conn_02x04_Odd_Even, Pin_Headers:Pin_Header_Angled_2x04_Pitch2.54mm, F.Cu at (152.5, 101.4)
- added R1: 160k, Resistors_SMD:R_0805, F.Cu at (69.1, 113.7)
- added R1: 160k, Resistors_SMD:R_0805, B.Cu at (209.1, 88.0)
- added R10: 330, Resistors_SMD:R_0805, F.Cu at (102.3, 98.4)
- added R10: 330, Resistors_SMD:R_0805, B.Cu at (219.0, 96.2)
- added R11: 10K, Resistors_SMD:R_0603, B.Cu at (29.1, 27.9)
- added R11: 10K, Resistors_SMD:R_0603, F.Cu at (153.0, 26.4)
- added R12: 10K, Resistors_SMD:R_0603, B.Cu at (30.9, 34.1)
- added R12: 10K, Resistors_SMD:R_0603, F.Cu at (154.8, 32.6)
- added R13: 10K, Resistors_SMD:R_0603, B.Cu at (30.9, 37.8)
- added R13: 10K, Resistors_SMD:R_0603, F.Cu at (154.7, 36.5)
- added R2: 30.1k, Resistors_SMD:R_0805, F.Cu at (65.8, 114.7)
- added R2: 30.1k, Resistors_SMD:R_0805, B.Cu at (212.4, 89.0)
- added R23: 330, Resistors_SMD:R_0603, B.Cu at (81.2, 115.0)
- added R23: 330, Resistors_SMD:R_0603, F.Cu at (196.9, 89.3)
- added R24: 180, Resistors_SMD:R_0603, B.Cu at (78.8, 114.9)
- added R24: 180, Resistors_SMD:R_0603, F.Cu at (199.3, 89.2)
- added R25: 1k, Resistors_SMD:R_0603, B.Cu at (84.2, 115.0)
- added R25: 1k, Resistors_SMD:R_0603, F.Cu at (193.9, 89.3)
- added R3: 100k, Resistors_SMD:R_0805, F.Cu at (63.6, 105.2)
- added R3: 100k, Resistors_SMD:R_0805, B.Cu at (214.6, 79.5)
- added R32: 0, Resistors_SMD:R_0805, B.Cu at (110.2, 82.0)
- added R32: 0, Resistors_SMD:R_0805, B.Cu at (233.8, 78.9)
- added R4: 63.4k, Resistors_SMD:R_0805, F.Cu at (60.6, 109.0)
- added R4: 63.4k, Resistors_SMD:R_0805, B.Cu at (190.5, 82.9)
- added R5: 160k, Resistors_SMD:R_0805, F.Cu at (80.4, 108.2)
- added R5: 160k, Resistors_SMD:R_0805, B.Cu at (197.7, 82.4)
- added R6: 51k, Resistors_SMD:R_0805, F.Cu at (76.9, 108.2)
- added R6: 51k, Resistors_SMD:R_0805, B.Cu at (201.2, 82.4)
- added R7: 100k, Resistors_SMD:R_0805, F.Cu at (75.4, 99.9)
- added R7: 100k, Resistors_SMD:R_0805, B.Cu at (202.8, 74.1)
- added R8: 56k, Resistors_SMD:R_0805, F.Cu at (72.8, 103.1)
- added R8: 56k, Resistors_SMD:R_0805, B.Cu at (205.4, 77.4)
- added R9: 330, Resistors_SMD:R_0805, F.Cu at (92.8, 97.9)
- added R9: 330, Resistors_SMD:R_0805, B.Cu at (228.5, 95.8)
- added REF**: SolderWirePad_1x01_SMD_5x10mm, Connector_Wire:SolderWirePad_1x01_SMD_5x10mm, F.Cu at (67.7, 85.2)
- added REF**: SolderWirePad_1x01_SMD_5x10mm, Connector_Wire:SolderWirePad_1x01_SMD_5x10mm, B.Cu at (193.7, 56.3)
- added REF**: MountingHole_3.2mm_M3, Mounting_Holes:MountingHole_3.2mm_M3, B.Cu at (231.3, 27.3)
- added REF**: SolderWirePad_1x01_SMD_5x10mm, Connector_Wire:SolderWirePad_1x01_SMD_5x10mm, B.Cu at (202.6, 56.3)
- added REF**: MountingHole_3.2mm_M3, Mounting_Holes:MountingHole_3.2mm_M3, F.Cu at (108.8, 116.1)
- added REF**: SolderWirePad_1x01_SMD_5x10mm, Connector_Wire:SolderWirePad_1x01_SMD_5x10mm, F.Cu at (76.6, 85.2)
- added REF**: MountingHole_3.2mm_M3, Mounting_Holes:MountingHole_3.2mm_M3, F.Cu at (28.8, 116.1)
- added REF**: MountingHole_3.2mm_M3, Mounting_Holes:MountingHole_3.2mm_M3, F.Cu at (32.6, 30.4)
- added REF**: SolderWirePad_1x01_SMD_5x10mm, Connector_Wire:SolderWirePad_1x01_SMD_5x10mm, F.Cu at (58.8, 85.2)
- added REF**: MountingHole_3.2mm_M3, Mounting_Holes:MountingHole_3.2mm_M3, F.Cu at (106.3, 30.4)
- added REF**: SolderWirePad_1x01_SMD_5x10mm, Connector_Wire:SolderWirePad_1x01_SMD_5x10mm, B.Cu at (184.8, 56.3)
- added REF**: MountingHole_3.2mm_M3, Mounting_Holes:MountingHole_3.2mm_M3, B.Cu at (157.6, 27.4)
- added SW1: SW_Push, Buttons_Switches_SMD:SW_SPST_B3U-1000P, F.Cu at (28.3, 28.1)
- added SW1: SW_Push, Buttons_Switches_SMD:SW_SPST_B3U-1000P, B.Cu at (152.2, 26.4)
- added SW2: SW_Push, Buttons_Switches_SMD:SW_SPST_B3U-1000P, F.Cu at (28.4, 32.8)
- added SW2: SW_Push, Buttons_Switches_SMD:SW_SPST_B3U-1000P, B.Cu at (152.3, 31.3)
- added SW3: SW_Push, Buttons_Switches_SMD:SW_SPST_B3U-1000P, F.Cu at (28.4, 37.7)
- added SW3: SW_Push, Buttons_Switches_SMD:SW_SPST_B3U-1000P, B.Cu at (152.3, 37.1)
- added U1: MPM3620, BusSimulator:QFN-20, F.Cu at (64.6, 110.5)
- added U1: MPM3620, BusSimulator:QFN-20, B.Cu at (213.6, 84.7)
- added U2: MPM3620, BusSimulator:QFN-20, F.Cu at (76.5, 104.4)
- added U2: MPM3620, BusSimulator:QFN-20, B.Cu at (201.7, 78.7)
- added U9: , Carrier-Board:mpcie-socket, B.Cu at (102.8, 59.0)
- added U9: , Carrier-Board:mpcie-socket, B.Cu at (226.2, 56.0)
- added m1: MountingHole_2.7mm_M2.5_Pad, Mounting_Holes:MountingHole_2.7mm_M2.5_Pad, F.Cu at (111.6, 45.1)
- added m1: MountingHole_2.7mm_M2.5_Pad, Mounting_Holes:MountingHole_2.7mm_M2.5_Pad, F.Cu at (111.6, 92.1)
- m1 (x2), m2: moved to B.Cu
- m2: moved to F.Cu
- moved m2 198.4 mm to (228.2, 89.1), turned to 180 degrees
- moved m2 142.9 mm to (35.8, 92.1)
- moved m1 46.9 mm to (152.4, 42.1), turned to 180 degrees
- moved m1 46.9 mm to (152.4, 89.1), turned to 180 degrees
- moved ? 14.1 mm to (238.5, 118.2)
Routing:
- net +3.3V: track 149.1 -> 525.7 mm
- net GPO2: track 311.6 -> 10.9 mm
- net WAKE1n: track 72.8 -> 303.7 mm, vias 2 -> 4
- net SPI_CLK: track 55.2 -> 265.1 mm, vias 3 -> 4
- net mCOM_5V_SBY: track 421.7 -> 264.5 mm
- net Net-(J4-Pad11): track 0.00 -> 154.6 mm
- net mCOM_12V: track 377.4 -> 223.3 mm, vias 8 -> 6
- net PWRBTNn: track 106.5 -> 216.3 mm, vias 5 -> 6
- net mCOM_TX: track 64.6 -> 165.6 mm, vias 2 -> 4
- net Net-(J5-Pad50): track 93.2 -> 0.00 mm, vias 4 -> 0
- net SYS_RESETn: track 88.2 -> 177.3 mm, vias 6 -> 8
- net GBE0_LINK1000#: track 78.0 -> 163.9 mm
- net GPO0: track 74.2 -> 150.5 mm, vias 2 -> 4
- net Net-(D7-Pad1): track 0.00 -> 73.2 mm, vias 3 -> 2
- net GPI2: track 65.9 -> 138.7 mm, vias 3 -> 4
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Other:
- outline, holes or cut-outs redrawn
