File: Carrier-Board-Mirroredv2/Carrier-Board.sch (KiCad schematic (older format))
At the start: 45 parts, among them J1 CONN_3-6318491-6, J10 Conn_02x03_Odd_Even, J2 Conn_01x0, J3 Conn_02x26_Odd_Even, J4 SI-51009-F, J5 Conn_02x26_Odd_Even, J6 Conn_01x03_Male, J7 Conn_01x03_Male, J8 Conn_01x06_Male, J9 Conn_02x04_Odd_Even, SW1 SW_Push, SW2 SW_Push, SW3 SW_Push, U1 MPM3620, U2 MPM3620, U9 MSATA-Socket

Commit message: USB schematic added
Added the USB addition for the carrier board into a schematic
Parts:
- added 100nF (x2), 10nF, 4.7uF: C, Capacitor_SMD:C_0603_1608Metric, symbol Device:C
- added D? (x2): LED, Diodes_SMD:D_1206, symbol Device:LED
- added L?: Ferrite_Bead, symbol Device:Ferrite_Bead
- added R (x2): 270, Resistors_SMD:R_0805, symbol Device:R
- added U?: FT232R, symbol New_Library:FT232R
- added U?: RS232LEVELCONVERTER, symbol New_Library:RS232LEVELCONVERTER
- added U?: DB9M, symbol New_Library:DB9M
- added U?: SHIELD, symbol New_Library:SHIELD
Connections:
- net labels added: GND
- wire segments 126 -> 201
Other:
- note added: "VCC"

Commit message: USB Schematic added
Added usb schematic, no footprints yet
Parts:
- G1: symbol Carrier-Board:LOGO -> BusSimulator:LOGO
- J1: symbol Carrier-Board:CONN_3-6318491-6 -> BusSimulator:CONN_3-6318491-6
- U1, U2: symbol Carrier-Board:MPM3620 -> BusSimulator:MPM3620
- U9: symbol Carrier-Board:MSATA-Socket -> BusSimulator:MSATA-Socket
Changed lines of the file:
@@
 $EndDescr
 $Comp
-L Carrier-Board:MPM3620 U1
+L BusSimulator:MPM3620 U1
 U 1 1 59F6A40E
 P 2500 2850
@@
 $EndComp
 $Comp
-L Power:GNDREF #PWR01
+L power:GNDREF #PWR01
 U 1 1 59F6A60F
 P 2325 1575
@@
 $EndComp
 $Comp
-L Power:GNDA #PWR02
+L power:GNDA #PWR02
 U 1 1 59F6AEAC
 P 3150 4000
@@
 $EndComp
 $Comp
-L Power:GNDA #PWR03
+L power:GNDA #PWR03
 U 1 1 59F6AF94
 P 1800 3250
@@
 $EndComp
 $Comp
-L Power:GNDA #PWR04
+L power:GNDA #PWR04
 U 1 1 59FA90DC
 P 3300 2000
@@
 $EndComp
 $Comp
-L Power:+5V #PWR05
+L power:+5V #PWR05
 U 1 1 59FAA2C5
 P 3150 2800
@@
 $EndComp
 $Comp
-L Carrier-Board:MPM3620 U2
+L BusSimulator:MPM3620 U2
 U 1 1 59FAACB4
 P 2450 5850
@@
 $EndComp
 $Comp
-L Power:GNDREF #PWR06
+L power:GNDREF #PWR06
 U 1 1 59FAACBA
 P 2275 4575
@@
 $EndComp
 $Comp
-L Power:GNDA #PWR07
+L power:GNDA #PWR07
 U 1 1 59FAACCC
 P 3100 7000
@@
 $EndComp
 $Comp
-L Power:GNDA #PWR08
+L power:GNDA #PWR08
 U 1 1 59FAACD8
 P 1750 6250
@@
 $EndComp
 $Comp
-L Power:GNDA #PWR09
+L power:GNDA #PWR09
 U 1 1 59FAACFB
 P 3250 5000
@@
 $EndComp
 $Comp
-L Power:+3.3V #PWR010
+L power:+3.3V #PWR010
 U 1 1 59FAAF36
 P 3100 5800
@@
 PCE3900CT-ND
 $Comp
-L Power:GNDREF #PWR011
+L power:GNDREF #PWR011
 U 1 1 59FACA7B
 P 3450 2550
@@
 $EndComp
 $Comp
-L Power:GNDREF #PWR012
+L power:GNDREF #PWR012
 U 1 1 59FACBAF
 P 3500 5500
@@
 $EndComp
 $Comp
-L Power:GNDREF #PWR013
+L power:GNDREF #PWR013
 U 1 1 59FACE9C
 P 3000 3550
@@
 $EndComp
 $Comp
-L Power:GNDREF #PWR014
+L power:GNDREF #PWR014
 U 1 1 59FAD007
 P 2250 1250
@@
 $EndComp
 $Comp
-L Power:GNDREF #PWR015
+L power:GNDREF #PWR015
 U 1 1 59FB82F0
 P 2250 4200
@@
 $EndComp
 $Comp
-L Power:GNDREF #PWR016
+L power:GNDREF #PWR016
 U 1 1 59FB843A
 P 2950 6550
@@
 $EndComp
 $Comp
-L Carrier-Board:CONN_3-6318491-6 J1
+L BusSimulator:CONN_3-6318491-6 J1
 U 1 1 5A03F4E1
 P 9450 4850
@@
 $EndComp
 $Comp
-L Carrier-Board:CONN_3-6318491-6 J1
+L BusSimulator:CONN_3-6318491-6 J1
 U 2 1 5A03F592
 P 10950 4850
@@
 $EndComp
 $Comp
-L Carrier-Board:CONN_3-6318491-6 J1
+L BusSimulator:CONN_3-6318491-6 J1
 U 3 1 5A03F60D
 P 12450 4850
@@
 $EndComp
 $Comp
-L Carrier-Board:CONN_3-6318491-6 J1
+L BusSimulator:CONN_3-6318491-6 J1
 U 4 1 5A03F69E
 P 13950 4850
@@
 $EndComp
 $Comp
-L Carrier-Board:CONN_3-6318491-6 J1
+L BusSimulator:CONN_3-6318491-6 J1
 U 5 1 5A03F72F
 P 15450 4850
@@
 mCOM_GND
 $Comp
-L Power:+12V #PWR017
+L power:+12V #PWR017
 U 1 1 5A040DA3
 P 2500 1500
@@
 $EndComp
 $Comp
-L Power:+12V #PWR018
+L power:+12V #PWR018
 U 1 1 5A040EAE
 P 2450 4500
@@
 $EndComp
 $Comp
-L Power:+12V #PWR019
+L power:+12V #PWR019
 U 1 1 5A0413FE
 P 1250 1850
@@
 $EndComp
 $Comp
-L Power:GNDREF #PWR020
+L power:GNDREF #PWR020
 U 1 1 5A04143A
 P 900 1750
@@
 +3.3V
 $Comp
-L Carrier-Board:LOGO G1
+L BusSimulator:LOGO G1
 U 1 1 5A0420BA
 P 10050 11050
@@
 $EndComp
 $Comp
-L Power:GNDREF #PWR021
+L power:GNDREF #PWR021
 U 1 1 5A08977E
 P 7000 2500
@@
 mCOM_12V
 $Comp
-L Carrier-Board:MSATA-Socket U9
+L BusSimulator:MSATA-Socket U9
 U 1 1 5A0BAE45
 P 2800 9300
@@
 +3.3V
 $Comp
-L Power:GNDREF #PWR022
+L power:GNDREF #PWR022
 U 1 1 5A0C1B77
 P 3700 8250
@@
 $EndComp
 $Comp
-L Power:GNDREF #PWR023
+L power:GNDREF #PWR023
 U 1 1 5A0C1C29
 P 3900 10650
@@
 $EndComp
 $Comp
-L Power:GNDREF #PWR024
+L power:GNDREF #PWR024
 U 1 1 5A0C1CDB
 P 4000 9450
@@
 $EndComp
 $Comp
-L Power:GNDREF #PWR025
+L power:GNDREF #PWR025
 U 1 1 5A0C1D8D
 P 4000 9050
@@
 $EndComp
 $Comp
-L Power:GNDREF #PWR026
+L power:GNDREF #PWR026
 U 1 1 5A0C1E3F
 P 4000 8750
@@
 $EndComp
 $Comp
-L Power:GNDREF #PWR027
+L power:GNDREF #PWR027
 U 1 1 5A0C1EF1
 P 4000 9850
@@
 SATA0_RX-
 $Comp
-L Power:GNDREF #PWR028
+L power:GNDREF #PWR028
 U 1 1 5A0C49FB
 P 1800 10400
@@
 $EndComp
 $Comp
-L Power:GNDREF #PWR029
+L power:GNDREF #PWR029
 U 1 1 5A0C4BAB
 P 1900 10050
@@
 Sata Connector\n
 $Comp
-L Power:GNDREF #PWR030
+L power:GNDREF #PWR030
 U 1 1 5A0C6A3D
 P 1450 8950
@@
 $EndComp
 $Comp
-L Power:GNDREF #PWR031
+L power:GNDREF #PWR031
 U 1 1 5A0C6D48
 P 1500 9350
@@
 $EndComp
 $Comp
-L Power:GNDREF #PWR032
+L power:GNDREF #PWR032
 U 1 1 5A0C77C7
 P 1600 8450
@@
 $EndComp
 $Comp
-L Power:GNDREF #PWR033
+L power:GNDREF #PWR033
 U 1 1 5A0DCFAA
 P 750 8350
@@
 $EndComp
 $Comp
-L Power:GNDREF #PWR034
+L power:GNDREF #PWR034
 U 1 1 5A0DD07C
 P 1100 9050
@@
 $EndComp
 $Comp
-L Power:GNDREF #PWR035
+L power:GNDREF #PWR035
 U 1 1 5A0DDC34
 P 4500 8450
@@
 $EndComp
 $Comp
-L Power:GNDREF #PWR036
+L power:GNDREF #PWR036
 U 1 1 5A0B68CF
 P 8750 1600
@@
 GBE0_CTREF(GND)
 $Comp
-L Power:GNDREF #PWR037
+L power:GNDREF #PWR037
 U 1 1 5A6D828B
 P 6150 5750
@@
 $EndComp
 $Comp
-L Power:GNDREF #PWR038
+L power:GNDREF #PWR038
 U 1 1 5A6D9E6B
 P 7250 5450
@@
 $EndComp
 $Comp
-L Power:GNDREF #PWR039
+L power:GNDREF #PWR039
 U 1 1 5A6DAA22
 P 7300 5050
@@
 $EndComp
 $Comp
-L Power:GNDREF #PWR040
+L power:GNDREF #PWR040
 U 1 1 5A6DB372
 P 5150 4750
@@
 Connection ~ 14400 2450
 $Comp
-L Power:GNDREF #PWR041
+L power:GNDREF #PWR041
 U 1 1 5A6EC603
 P 14350 1300
@@
 $EndComp
 $Comp
-L Power:GNDREF #PWR042
+L power:GNDREF #PWR042
 U 1 1 5A6EC92F
 P 14400 2100
@@
 $EndComp
 $Comp
-L Power:GNDREF #PWR043
+L power:GNDREF #PWR043
 U 1 1 5A6ECB43
 P 14400 3000

Commit message: USB Port Schematic Added
added the USB port schematic
Parts:
- removed 100nF (x2), 10nF, 4.7uF: C, Capacitor_SMD:C_0603_1608Metric, symbol Device:C
- removed D? (x2): LED, Diodes_SMD:D_1206, symbol Device:LED
- removed L?: Ferrite_Bead, symbol Device:Ferrite_Bead
- removed R (x2): 270, Resistors_SMD:R_0805, symbol Device:R
- removed U?: FT232R, symbol New_Library:FT232R
- removed U?: RS232LEVELCONVERTER, symbol New_Library:RS232LEVELCONVERTER
- removed U?: DB9M, symbol New_Library:DB9M
- removed U?: SHIELD, symbol New_Library:SHIELD
- added C10, C5, C6: .1uF, Capacitor_SMD:C_0603_1608Metric, symbol Device:C
- added C11, C12, C8: .33uF, Capacitor_SMD:C_0603_1608Metric, symbol Device:C
- added C7: 47nF, Capacitor_SMD:C_0603_1608Metric, symbol Device:C
- added C9: 4.7uF, Capacitor_SMD:C_0603_1608Metric, symbol Device:C
- added D1: SP0502BAJT, Package_TO_SOT_SMD:SOT-323_SC-70, symbol Power_Protection:SP0502BAJT
- added D2, D3: LED, symbol Device:LED
- added J11: USB_B_Micro, symbol Connector:USB_B_Micro
- added R14: 10K, symbol Device:R
- added R15: 4.7K, symbol Device:R
- added R? (x2): R, symbol Device:R
- added U?: MAX3221, symbol Interface_UART:MAX3221
- added U?: FT232RQ, symbol USB:FT232RQ
Connections:
- net labels added: RXD, Reset#, TXD
- net labels removed: GND
- wire segments 201 -> 209
- no-connect marks 0 -> 18
Other:
- note added: "USB to RS232"
- note added: "polarized +"
- note added: "polarized -"
- note removed: "VCC"

Commit message: Revised Mirrored Board
Complete mirrored board with traces (Minus micro USB port)
Parts:
- J11: footprint (none) -> Connector_USB:USB_Micro-B_Molex-105017-0001
- U?: footprint (none) -> Package_SO:SSOP-16_4.4x5.2mm_P0.65mm
- U?: footprint (none) -> Package_SO:SSOP-28_3.9x9.9mm_P0.635mm
Changed lines of the file:
@@
 F 0 "U?" H 6450 6328 50  0000 C CNN
 F 1 "MAX3221" H 6450 6237 50  0000 C CNN
-F 2 "" H 6500 5250 50  0001 C CIN
+F 2 "Package_SO:SSOP-16_4.4x5.2mm_P0.65mm" H 6500 5250 50  0001 C CIN
 F 3 "http://www.ti.com/lit/ds/symlink/max3221.pdf" H 6450 6200 50  0001 C CNN
 	1    6450 5250
@@
 F 0 "U?" H 7341 7796 50  0000 L CNN
 F 1 "FT232RQ" H 7341 7705 50  0000 L CNN
-F 2 "" H 6650 7750 50  0001 C CNN
+F 2 "Package_SO:SSOP-28_3.9x9.9mm_P0.635mm" H 6650 7750 50  0001 C CNN
 F 3 "" H 6650 7750 50  0001 C CNN
 	1    6800 7800
@@
 F 0 "J11" H 6600 10700 50  0000 L CNN
 F 1 "USB_B_Micro" H 6450 10600 50  0000 L CNN
-F 2 "" H 6800 10150 50  0001 C CNN
+F 2 "Connector_USB:USB_Micro-B_Molex-105017-0001" H 6800 10150 50  0001 C CNN
 F 3 "~" H 6800 10150 50  0001 C CNN
 	1    6650 10200
